File: SpookyCastle/node-Atmega328-board/untitled.brd (EAGLE design)
At the start: 49.7 x 36 mm, 23 parts, among them IC2 MEGA48/88/168-AU

Commit message: whole buncha changes
Parts:
- added U$1: OSHW-LOGOM, SparkFun - Copy:OSHW-LOGO-M
- C5: value 1uF -> 0.1uF
- moved C1 0.40 mm to (21.5, 43.9)
Routing:
- net N$14: track 9.95 -> 7.53 mm
- net DI: track 25.1 -> 23.7 mm
- net RO: track 16.4 -> 15.2 mm
- net P27: track 12.5 -> 11.3 mm
- net N$5: track 22.5 -> 23.2 mm
- net GND: vias 17 -> 20
Other:
- board text added: "9-36V+"
- board text added: "Bus GND"
- board text added: "CC-BY-SA"
- board text added: "In the dark halls many things dwell"
- board text added: "Keep your wits, all shall be well..."
- board text added: "RS485 A"
- board text added: "RS485 B"
- board text added: "SpookyCastle I/O Board"
- board text added: "Version 1 By Daniel Black"
